Commit message: [add]:在gazebo世界模型中加载机器人

File: products/cpp/fishbot_desc_ws/src/fishbot_description/urdf/fishbot/actuator/caster.urdf.xacro (robot description, xacro)
@@ -3,4 +3,7 @@
 <!--声明驱动轮模块-->
 <xacro:macro name="caster_xacro" params="caster_name xyz">
+    <gazebo reference="${caster_name}_caster_link">
+        <material>Gazebo/Yellow</material>
+    </gazebo>
     <link name="${caster_name}_caster_link">
     <!--驱动轮子的身体部分-->

File: products/cpp/fishbot_desc_ws/src/fishbot_description/urdf/fishbot/actuator/wheel.urdf.xacro (robot description, xacro)
@@ -3,4 +3,10 @@
 <!--声明驱动轮模块-->
 <xacro:macro name="wheel_xacro" params="wheel_name xyz">
+    <gazebo reference="${wheel_name}_wheel_link">
+        <material>Gazebo/Yellow</material>
+    </gazebo>
+    <gazebo reference="${wheel_name}_wheel_link">
+        <material>Gazebo/Yellow</material>
+    </gazebo>
     <link name="${wheel_name}_wheel_link">
     <!--驱动轮子的身体部分-->

File: products/cpp/fishbot_desc_ws/src/fishbot_description/urdf/fishbot/sensor/camera.urdf.xacro (robot description, xacro)
@@ -3,4 +3,7 @@
 <!--声明base模块-->
 <xacro:macro name="camera_xacro" params="xyz">
+    <gazebo reference="camera_link">
+        <material>Gazebo/Green</material>
+    </gazebo>
     <link name="camera_link">
     <!--机器人的身体部分-->

File: products/cpp/fishbot_desc_ws/src/fishbot_description/urdf/fishbot/sensor/imu.urdf.xacro (robot description, xacro)
@@ -2,4 +2,7 @@
 <robot xmlns:xacro="http://www.ros.org/wiki/xacro">
 <xacro:macro name="imu_xacro" params="xyz">
+    <gazebo reference="imu_link">
+        <material>Gazebo/Black</material>
+    </gazebo>
     <link name="imu_link">
     <!--imu惯性传感器的身体部分-->

File: products/cpp/fishbot_desc_ws/src/fishbot_description/urdf/fishbot/sensor/laser.urdf.xacro (robot description, xacro)
@@ -3,4 +3,11 @@
 <!--声明base模块-->
 <xacro:macro name="laser_xacro" params="xyz">
+    <!--在gazebo中将颜色改为黑色-->
+    <gazebo reference="laser_cylinder_link">
+        <material>Gazebo/Black</material>
+    </gazebo>
+    <gazebo reference="laser_link">
+        <material>Gazebo/Black</material>
+    </gazebo>
     <!-- 雷达支撑杆 -->
     <link name="laser_cylinder_link">
